Commit message: add multiple belt in model

File: ur_gazebo/urdf/ur5e_link_d405_robotiq.xacro (robot description, xacro)
@@ -74,5 +74,5 @@
     <origin xyz="0 0 0" rpy="0 0 0"/>
   </joint>
-  <!--PU Belt-->
+  <!--PU Belt1-->
   <xacro:include filename="$(find belt12mm_description)/urdf/belt12mm.xacro"/>
   <xacro:belt12mm parent="base_link" prefix="belt12mm_">
@@ -83,4 +83,22 @@
           <child link="belt12mm_base_link"/>
           <origin xyz="0.5 0.0 0" rpy="1.57 0 1.57"/>
+  </joint>
+  <xacro:belt12mm parent="base_link" prefix="belt12mm_2_">
+    <origin xyz="0.0 0.0 0.0" rpy="0.0 0.0 0.0"/>
+  </xacro:belt12mm>
+  <joint name="belt12mm_2_joint" type="fixed">
+          <parent link="base_link"/>
+          <child link="belt12mm_2_base_link"/>
+          <origin xyz="0.4 0.1 0" rpy="1.57 0 1.57"/>
+  </joint>
+  <!--PU Belt2-->
+  <xacro:include filename="$(find belt10mm_description)/urdf/belt10mm.xacro"/>
+  <xacro:belt12mm parent="base_link" prefix="belt10mm_">
+    <origin xyz="0.0 0.0 0.0" rpy="0.0 0.0 0.0"/>
+  </xacro:belt12mm>
+  <joint name="belt10mm_joint" type="fixed">
+          <parent link="base_link"/>
+          <child link="belt10mm_base_link"/>
+          <origin xyz="0.3 0.1 0" rpy="1.57 0 1.57"/>
   </joint>
   <!--Connect Camera Link-->

Commit message: [ok] workable

File: ur_gazebo/urdf/ur5e_link_d405_robotiq.xacro (robot description, xacro)
@@ -82,5 +82,5 @@
           <parent link="base_link"/>
           <child link="belt12mm_base_link"/>
-          <origin xyz="0.5 0.0 0" rpy="1.57 0 1.57"/>
+          <origin xyz="0.55 0.08 0" rpy="1.57 0 1.57"/>
   </joint>
   <xacro:belt12mm parent="base_link" prefix="belt12mm_2_">
@@ -90,5 +90,5 @@
           <parent link="base_link"/>
           <child link="belt12mm_2_base_link"/>
-          <origin xyz="0.4 0.1 0" rpy="1.57 0 1.57"/>
+          <origin xyz="0.5 0.18 0.02" rpy="1.57 0 1.57"/>
   </joint>
   <!--PU Belt2-->
@@ -100,5 +100,5 @@
           <parent link="base_link"/>
           <child link="belt10mm_base_link"/>
-          <origin xyz="0.3 0.1 0" rpy="1.57 0 1.57"/>
+          <origin xyz="0.25 -0.03 0" rpy="1.57 0 1.57"/>
   </joint>
   <!--Connect Camera Link-->

Commit message: belt rotate in 3D space

File: ur_gazebo/urdf/ur5e_link_d405_robotiq.xacro (robot description, xacro)
@@ -82,5 +82,6 @@
           <parent link="base_link"/>
           <child link="belt12mm_base_link"/>
-          <origin xyz="0.55 0.08 0" rpy="1.57 0 1.57"/>
+          <!-- <origin xyz="0.55 0.08 0" rpy="1.57 0 1.57"/> -->
+          <origin xyz="0.55 0.08 0.1" rpy="0.5 0 1.57"/>
   </joint>
   <xacro:belt12mm parent="base_link" prefix="belt12mm_2_">
@@ -90,5 +91,6 @@
           <parent link="base_link"/>
           <child link="belt12mm_2_base_link"/>
-          <origin xyz="0.5 0.18 0.02" rpy="1.57 0 1.57"/>
+          <!-- <origin xyz="0.5 0.18 0.02" rpy="1.57 0 1.57"/> -->
+          <origin xyz="0.5 0.18 0.1" rpy="0.5 0 1.57"/>
   </joint>
   <!--PU Belt2-->
@@ -100,5 +102,6 @@
           <parent link="base_link"/>
           <child link="belt10mm_base_link"/>
-          <origin xyz="0.25 -0.03 0" rpy="1.57 0 1.57"/>
+          <!-- <origin xyz="0.25 -0.03 0.1" rpy="1.57 0 1.57"/> -->
+          <origin xyz="0.25 -0.03 0.1" rpy="0.5 0 1.57"/>
   </joint>
   <!--Connect Camera Link-->
